File: Eagle Files/round board.sch (EAGLE design)
At the start: 7 parts

Commit message: Moved AS5600 footprint to center of board (v1.1)
Removed pull-up resistors
Parts:
- removed R1, R2: 4.7K, SparkFun-Resistors:4.7KOHM-1/10W-1%(0603)
Connections:
- net SCL: no longer R2.1
- net SDA: no longer R1.2
- net VDD5V: no longer R1.1, R2.2
Changed lines of the file:
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@@
 <part name="C1" library="SparkFun-Capacitors" deviceset="1.0UF-16V-10%(0603)" device="" value="1.0uF"/>
 <part name="C2" library="SparkFun-Capacitors" deviceset="0.1UF-25V(+80/-20%)(0603)" device="" value="0.1uF"/>
-<part name="R1" library="SparkFun-Resistors" deviceset="4.7KOHM-1/10W-1%(0603)" device="" value="4.7K"/>
-<part name="R2" library="SparkFun-Resistors" deviceset="4.7KOHM-1/10W-1%(0603)" device="" value="4.7K"/>
 <part name="D1" library="SparkFun-DiscreteSemi" deviceset="DIODE" device="BAS16" value="250mA/100V"/>
 </parts>
@@
 <instance part="C1" gate="G$1" x="25.4" y="40.64"/>
 <instance part="C2" gate="G$1" x="20.32" y="43.18" rot="R180"/>
-<instance part="R1" gate="G$1" x="81.28" y="30.48" rot="R90"/>
-<instance part="R2" gate="G$1" x="81.28" y="50.8" rot="R90"/>
 <instance part="D1" gate="G$1" x="109.22" y="30.48" rot="R270"/>
 </instances>
@@
 <wire x1="20.32" y1="50.8" x2="20.32" y2="45.72" width="0.1524" layer="91"/>
 <junction x="25.4" y="50.8"/>
-</segment>
-<segment>
-<pinref part="R2" gate="G$1" pin="2"/>
-<wire x1="81.28" y1="55.88" x2="88.9" y2="55.88" width="0.1524" layer="91"/>
-<label x="88.9" y="55.88" size="1.778" layer="95" xref="yes"/>
-</segment>
-<segment>
-<pinref part="R1" gate="G$1" pin="1"/>
-<wire x1="81.28" y1="25.4" x2="81.28" y2="17.78" width="0.1524" layer="91"/>
-<label x="81.28" y="17.78" size="1.778" layer="95" rot="R270" xref="yes"/>
 </segment>
 <segment>
@@
 <segment>
 <pinref part="U$1" gate="G$1" pin="SCL"/>
-<wire x1="73.66" y1="45.72" x2="81.28" y2="45.72" width="0.1524" layer="91"/>
+<wire x1="73.66" y1="45.72" x2="83.82" y2="45.72" width="0.1524" layer="91"/>
 <label x="83.82" y="45.72" size="1.778" layer="95" xref="yes"/>
-<pinref part="R2" gate="G$1" pin="1"/>
-<wire x1="81.28" y1="45.72" x2="83.82" y2="45.72" width="0.1524" layer="91"/>
-<junction x="81.28" y="45.72"/>
 </segment>
 <segment>
@@
 <segment>
 <pinref part="U$1" gate="G$1" pin="SDA"/>
-<wire x1="73.66" y1="40.64" x2="81.28" y2="40.64" width="0.1524" layer="91"/>
+<wire x1="73.66" y1="40.64" x2="83.82" y2="40.64" width="0.1524" layer="91"/>
 <label x="83.82" y="40.64" size="1.778" layer="95" xref="yes"/>
-<junction x="81.28" y="40.64"/>
-<wire x1="81.28" y1="40.64" x2="83.82" y2="40.64" width="0.1524" layer="91"/>
-<pinref part="R1" gate="G$1" pin="2"/>
-<wire x1="81.28" y1="40.64" x2="81.28" y2="35.56" width="0.1524" layer="91"/>
 </segment>
 <segment>
